File: pcb/eink_driver.kicad_pcb (KiCad board)
At the start: 4 copper layers, 0 parts

Commit message: Tied physical components to layout components and created initial pcb file
Parts:
- added D1: D_Schottky, Diode_SMD:D_SMA, F.Cu at (126.8, 67.8)
- added D2: D_Schottky, Diode_SMD:D_SMA, F.Cu at (111.5, 129.5)
- added D3: D_Schottky, Diode_SMD:D_SMA, F.Cu at (121.2, 72.7)
- added D4: D_Schottky, Diode_SMD:D_SMA, F.Cu at (108.5, 110.0)
- added J2: Conn_02x08_Counter_Clockwise, Connector_PinSocket_2.54mm:PinSocket_2x08_P2.54mm_Vertical, F.Cu at (93.5, 121.7)
- added J3: 3.3V Jumper, Connector_PinHeader_2.54mm:PinHeader_1x02_P2.54mm_Vertical, F.Cu at (139.1, 122.0)
- added JP1: P10 NC, Jumper:SolderJumper-2_P1.3mm_Open_Pad1.0x1.5mm, B.Cu at (160.7, 113.1)
- added JP2: P9 NC, Jumper:SolderJumper-2_P1.3mm_Open_Pad1.0x1.5mm, B.Cu at (160.6, 110.2)
- added JP3: SolderJumper_3_Bridged12, Jumper:SolderJumper-3_P1.3mm_Bridged12_Pad1.0x1.5mm, F.Cu at (136.5, 66.0)
- added JP4: SolderJumper_3_Bridged12, Jumper:SolderJumper-3_P1.3mm_Bridged12_Pad1.0x1.5mm, F.Cu at (103.0, 136.5)
- added JP5: SolderJumper_3_Bridged12, Jumper:SolderJumper-3_P1.3mm_Bridged12_Pad1.0x1.5mm, F.Cu at (123.3, 100.4)
- added R1: 10k, Resistor_SMD:R_0603_1608Metric, F.Cu at (159.4, 103.4)
- added R10: 100k, Resistor_SMD:R_0603_1608Metric, F.Cu at (116.5, 134.0)
- added R11: 100k, Resistor_SMD:R_0603_1608Metric, F.Cu at (119.7, 134.0)
- added R12: 1k, Resistor_SMD:R_0603_1608Metric, F.Cu at (117.7, 70.0)
- added R13: 1k, Resistor_SMD:R_0603_1608Metric, F.Cu at (126.7, 62.2)
- added R14: 1k, Resistor_SMD:R_0603_1608Metric, F.Cu at (111.5, 135.0)
- added R15: 10k, Resistor_SMD:R_0603_1608Metric, F.Cu at (116.2, 67.7)
- added R16: 16k, Resistor_SMD:R_0603_1608Metric, F.Cu at (121.5, 66.0)
- added R17: 10k, Resistor_SMD:R_0603_1608Metric, F.Cu at (125.2, 109.3)
- added R18: 10k, Resistor_SMD:R_0603_1608Metric, F.Cu at (133.3, 99.9)
- added R19: 83k, Resistor_SMD:R_0603_1608Metric, F.Cu at (129.5, 106.8)
- added R2: 10k, Resistor_SMD:R_0603_1608Metric, F.Cu at (139.2, 65.0)
- added R20: 5k, Resistor_SMD:R_0603_1608Metric, F.Cu at (137.6, 102.4)
- added R3: 10k, Resistor_SMD:R_0603_1608Metric, F.Cu at (139.2, 67.0)
- added R4: 10k, Resistor_SMD:R_0603_1608Metric, F.Cu at (102.0, 132.5)
- added R5: 10k, Resistor_SMD:R_0603_1608Metric, F.Cu at (103.5, 132.5)
- added R6: 12k, Resistor_SMD:R_0603_1608Metric, F.Cu at (120.5, 131.5)
- added R7: 140k, Resistor_SMD:R_0603_1608Metric, F.Cu at (118.0, 67.7)
- added R8: 100k, Resistor_SMD:R_0603_1608Metric, F.Cu at (124.0, 65.3)
- added R9: 100k, Resistor_SMD:R_0603_1608Metric, F.Cu at (121.5, 64.5)
- added RV1: 10k, Potentiometer_SMD:Potentiometer_Bourns_3269W_Vertical, F.Cu at (150.3, 127.8)
- added U1: ED060SC4, Connector_FFC-FPC:Molex_502250-3991_2Rows-39Pins-1MP_P0.60mm_Horizontal, F.Cu at (170.6, 111.8)
- added U2: R1283x, ATL:SON50P300X270X60-13N, F.Cu at (121.5, 68.7)
- added U3: R1283x, ATL:SON50P300X270X60-13N, F.Cu at (117.0, 129.5)
- added U4: LM2611xMF, Package_TO_SOT_SMD:SOT-23-5, F.Cu at (128.8, 100.8)
- added U5: AP3012, Package_TO_SOT_SMD:SOT-23-5, F.Cu at (112.7, 114.5)
