File: pcb/eink_driver.kicad_sch (KiCad schematic)
At the start: 0 parts

Commit message: Progress
Parts:
- added J?: Power Breakout, symbol Connector_Generic:Conn_01x06
- added J?: Conn_02x08_Counter_Clockwise, symbol Connector_Generic:Conn_02x08_Counter_Clockwise
- added J?: 3.3V Jumper, symbol Connector_Generic:Conn_01x02
- added J?: Conn_01x03, symbol Connector_Generic:Conn_01x03
- added JP?: P10 NC, symbol Jumper:SolderJumper_2_Open
- added JP?: P9 NC, symbol Jumper:SolderJumper_2_Open
- added R?: 10k, symbol Device:R_Small_US
- added RV?: 10k, symbol Device:R_Potentiometer_Trim_US
- added U?: ED060SC4, Connector_FFC-FPC:Molex_502250-3991_2Rows-39Pins-1MP_P0.60mm_Horizontal, symbol ATL:ED060SC4
Connections:
- new net: JP?.2 (B), U?.10 (NC)
- new net: R?.2, RV?.1, U?.22 (VCOM)
- new net: JP?.2 (B), U?.9 (NC)
- new net: J?.1 (Pin_1), J?.2 (Pin_2)
- new net +15V: J?.2 (Pin_2), U?.2 (VPOS)
- new net +22V: J?.3 (Pin_3), U?.23 (GVDD)
- new net +3V3: J?.1 (Pin_1), J?.3 (Pin_3), JP?.1 (A), U?.30 (U1CE2), U?.35 (U2CE2), U?.36 (U2CE1), U?.4 (VDD), U?.8 (SHR)
- new net -15V: J?.5 (Pin_5), R?.1, U?.1 (VNEG)
- new net -20V: J?.4 (Pin_4), U?.24 (GVEE)
- new net CKV: J?.7 (Pin_7), U?.33 (U1CKV), U?.38 (U2CKV)
- new net CL: J?.1 (Pin_1), U?.5 (CL)
- new net D0: J?.16 (Pin_16)
- new net D1: J?.15 (Pin_15)
- new net D2: J?.14 (Pin_14)
- new net D3: J?.13 (Pin_13)
- new net D4: J?.12 (Pin_12)
- new net D5: J?.11 (Pin_11)
- new net D6: J?.10 (Pin_10)
- new net D7: J?.9 (Pin_9)
- new net GMODE: J?.5 (Pin_5), U?.27 (GMODE2), U?.28 (GMODE1)
- new net GND: J?.6 (Pin_6), J?.8 (Pin_8), JP?.1 (A), RV?.2, U?.29 (RL), U?.3 (VSS), U?.31 (U1CE1), U?.34 (VBORDER)
- new net LE: J?.2 (Pin_2), U?.6 (LE)
- new net OE: J?.3 (Pin_3), U?.7 (OE)
- new net SPH: J?.4 (Pin_4), U?.11 (SPH)
- new net SPV: J?.6 (Pin_6), U?.32 (U1SPV), U?.37 (U2SPV)
- new net VD: J?.1 (Pin_1)
- new net VDD: J?.2 (Pin_2)
- no-connect marks 0 -> 1
Other:
- added sheet Voltage Regulators (untitled.kicad_sch)

Commit message: Tied physical components to layout components and created initial pcb file
Parts:
- J2: renamed from J?; footprint (none) -> Connector_PinSocket_2.54mm:PinSocket_2x08_P2.54mm_Vertical
- J3: renamed from J?; footprint (none) -> Connector_PinHeader_2.54mm:PinHeader_1x02_P2.54mm_Vertical
- JP1, JP2: renamed from JP?; footprint (none) -> Jumper:SolderJumper-2_P1.3mm_Open_Pad1.0x1.5mm
- R1: renamed from R?; footprint (none) -> Resistor_SMD:R_0603_1608Metric
- RV1: renamed from RV?; footprint (none) -> Potentiometer_SMD:Potentiometer_Bourns_3269W_Vertical
- gave numbers to parts that had none: 3
